File: stm32f030_adc/power-mcu.kicad_sch (KiCad schematic)
At the start: 28 parts, among them U1 STM32F103C6Tx, U2 AMS1117-3.3, X1 USB_B_Micro, Y2 8 MHz

Commit message: INTERMEDIATE
Parts:
- removed R3: 0, Resistor_THT:R_Axial_DIN0207_L6.3mm_D2.5mm_P10.16mm_Horizontal, symbol pspice:R
Changed lines of the file:
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@@
 	)
 	(junction
-		(at 83.82 146.05)
-		(diameter 0)
-		(color 0 0 0 0)
-	)
-	(junction
 		(at 207.01 82.55)
 		(diameter 0)
@@
 	(wire
 		(pts
-			(xy 68.58 139.7) (xy 68.58 146.05)
-		)
-		(stroke
-			(width 0)
-			(type default)
-		)
-	)
-	(wire
-		(pts
 			(xy 121.92 59.69) (xy 128.27 59.69)
 		)
@@
 	(wire
 		(pts
-			(xy 83.82 146.05) (xy 83.82 154.94)
-		)
-		(stroke
-			(width 0)
-			(type default)
-		)
-	)
-	(wire
-		(pts
 			(xy 185.42 80.01) (xy 187.96 80.01)
 		)
@@
 	(wire
 		(pts
-			(xy 81.28 139.7) (xy 83.82 139.7)
-		)
-		(stroke
-			(width 0)
-			(type default)
-		)
-	)
-	(wire
-		(pts
 			(xy 187.96 88.9) (xy 187.96 86.36)
 		)
@@
 	(wire
 		(pts
-			(xy 68.58 146.05) (xy 83.82 146.05)
-		)
-		(stroke
-			(width 0)
-			(type default)
-		)
-	)
-	(wire
-		(pts
 			(xy 207.01 86.36) (xy 219.71 86.36)
 		)
@@
 	(wire
 		(pts
-			(xy 83.82 139.7) (xy 83.82 146.05)
+			(xy 83.82 146.05) (xy 83.82 154.94)
 		)
 		(stroke
@@
 		)
 	)
+	(wire
+		(pts
+			(xy 68.58 146.05) (xy 83.82 146.05)
+		)
+		(stroke
+			(width 0)
+			(type default)
+		)
+	)
 	(text "Full speed USB device"
 		(exclude_from_sim no)
@@
 	(label "USART_1_RX"
 		(at 198.12 121.92 180)
-		(fields_autoplaced yes)
 		(effects
 			(font
@@
 	(label "USB_D-"
 		(at 77.47 50.8 0)
-		(fields_autoplaced yes)
 		(effects
 			(font
@@
 	(label "SWD_IO"
 		(at 198.12 129.54 180)
-		(fields_autoplaced yes)
 		(effects
 			(font
@@
 	(label "USART_1_TX"
 		(at 198.12 119.38 180)
-		(fields_autoplaced yes)
 		(effects
 			(font
@@
 	(label "USB_D+"
 		(at 77.47 48.26 0)
-		(fields_autoplaced yes)
 		(effects
 			(font
@@
 	(label "USB_D-"
 		(at 198.12 124.46 180)
-		(fields_autoplaced yes)
 		(effects
 			(font
@@
 	(label "SWD_CLK"
 		(at 198.12 132.08 180)
-		(fields_autoplaced yes)
 		(effects
 			(font
@@
 	(label "USB_D+"
 		(at 198.12 127 180)
-		(fields_autoplaced yes)
 		(effects
 			(font
@@
 		(shape input)
 		(at 187.96 99.06 0)
-		(fields_autoplaced yes)
 		(effects
 			(font
@@
 					(unit 1)
 				)
-			)
-		)
-	)
-	(symbol
-		(lib_id "pspice:R")
-		(at 74.93 139.7 270)
-		(mirror x)
-		(unit 1)
-		(exclude_from_sim no)
-		(in_bom yes)
-		(on_board yes)
-		(dnp no)
-		(property "Reference" "R3"
-			(at 74.93 133.35 90)
-			(effects
-				(font
-					(size 1.27 1.27)
-				)
-			)
-		)
-		(property "Value" "0"
-			(at 74.93 135.89 90)
-			(effects
-				(font
-					(size 1.27 1.27)
-				)
-			)
-		)
-		(property "Footprint" "Resistor_THT:R_Axial_DIN0207_L6.3mm_D2.5mm_P10.16mm_Horizontal"
-			(at 74.93 139.7 0)
-			(effects
-				(font
-					(size 1.27 1.27)
-				)
-				(hide yes)
-			)
-		)
-		(property "Datasheet" "~"
-			(at 74.93 139.7 0)
-			(effects
-				(font
-					(size 1.27 1.27)
-				)
-				(hide yes)
-			)
-		)
-		(property "Description" ""
-			(at 74.93 139.7 0)
-			(effects
-				(font
-					(size 1.27 1.27)
-				)
-				(hide yes)
-			)
-		)
-		(pin "1"
-		)
-		(pin "2"
-		)
-		(instances
-			(project "stm32f030_adc"
-				(path "/85629656-c73b-4e1f-b8e8-4366f4b01266/961be52f-ca6e-47db-97af-a75ea0ab8933"
-					(reference "R3")
-					(unit 1)
-				)
