File: stm32f030_adc/stm32f030_adc.kicad_pcb (KiCad board)
At the start: 2 copper layers, 50 x 93.5 mm, 47 parts, among them Q1 BC337, U1 STM32F103C6Tx, U2 AMS1117-3.3, X1 USB_B_Micro, Y2 8 MHz

Commit message: INTERMEDIATE
Parts:
- removed R3: 0, Resistor_THT:R_Axial_DIN0207_L6.3mm_D2.5mm_P10.16mm_Horizontal
- U1: moved to B.Cu
- moved R9 103.7 mm to (228.1, 94.0), turned to 180 degrees
- moved C17 99.6 mm to (218.2, 81.5), turned to 0 degrees
- moved R18 96.2 mm to (197.5, 79.5), turned to 180 degrees
- moved R16 93.4 mm to (197.5, 76.5), turned to 180 degrees
- moved R14 90.6 mm to (217.8, 100.0)
- moved R15 85.0 mm to (215.5, 71.0)
- moved R12 80.5 mm to (217.8, 97.0), turned to 0 degrees
- moved R8 75.5 mm to (215.6, 68.0), turned to 0 degrees
- moved Q1 75.4 mm to (204.7, 87.0), turned to 0 degrees
- moved R22 74.7 mm to (215.3, 74.0), turned to 0 degrees
- moved X1 71.4 mm to (205.6, 109.2)
- moved R19 69.9 mm to (187.8, 93.5)
- moved Y2 68.2 mm to (213.0, 101.0), turned to 90 degrees
- moved R6 65.1 mm to (218.0, 103.0), turned to 0 degrees
- moved C1 64.6 mm to (200.5, 72.0), turned to 90 degrees
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Routing:
- net GNDREF: track 367.2 -> 3.71 mm
- net +3V3: track 293.7 -> 12.0 mm
- net /Electret AMP/MIC_AMP_OUT: track 94.5 -> 0.00 mm
- net Net-(Q1-C): track 57.5 -> 0.00 mm
- net Net-(Q1-B): track 47.8 -> 0.00 mm
- net /Power and MCU/USB_D-: track 37.7 -> 0.00 mm
- net Net-(Q1-E): track 36.6 -> 0.00 mm
- net /Power and MCU/USB_D+: track 44.2 -> 11.4 mm
- net Net-(X1-D+): track 26.9 -> 0.00 mm
- net Net-(X1-D-): track 24.2 -> 0.00 mm
- net 5V_USB: track 25.2 -> 8.73 mm
- net Net-(U1-NRST): track 16.4 -> 0.00 mm
- net Net-(MK1-+): track 15.2 -> 0.00 mm
- net Net-(U1-BOOT0): track 12.6 -> 0.00 mm
- net Net-(U2-ADJ): track 9.39 -> 21.3 mm
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Other:
- board outline removed
